Commit message: fix(urdf): close 3 sensor joints with </joint> (was </link>)
Found while validating URDF with xacro: three sensor joints
(camera_front, ir_left, ir_right) were closed with </link> instead
of </joint>. This is a copy-paste error from a draft where all
sections were the same shape.

xacro expansion now passes:
- 14 links (base + 4 wheels + 5 arm + 2 cam + 2 IR)
- 21 joints (4 wheel continuous + 1 arm_base fixed + 2 prismatic
  + 1 rotate + 1 grip + 4 sensor fixed + 8 ros2_control command/state)
- 1 ros2_control block (MC602 system interface)

Verified locally with `xacro vehicle_wbt.urdf.xacro > /tmp/...urdf`.

Co-Authored-By: Claude <noreply@anthropic.com>

File: ros2_ws/src/vehicle_wbt_platform_cpp/urdf/vehicle_wbt.urdf.xacro (robot description, xacro)
@@ -172,5 +172,5 @@
     <child link="camera_front_link"/>
     <origin xyz="${chassis_length/2 - 0.01} 0 ${chassis_height/2}" rpy="0 0 0"/>
-  </link>
+  </joint>
   <!-- Side camera (P8 /dev/cam1) -->
   <link name="camera_side_link"/>
@@ -186,5 +186,5 @@
     <child link="ir_left_link"/>
     <origin xyz="0 ${chassis_width/2 - 0.02} ${chassis_height/2}" rpy="0 0 0"/>
-  </link>
+  </joint>
   <link name="ir_right_link"/>
   <joint name="ir_right_joint" type="fixed">
@@ -192,5 +192,5 @@
     <child link="ir_right_link"/>
     <origin xyz="0 ${-chassis_width/2 + 0.02} ${chassis_height/2}" rpy="0 0 0"/>
-  </link>
+  </joint>
   <!-- ================= ros2_control hardware interface ================= -->
   <ros2_control name="MC602" type="system">
